Commit message: The hardware interface has problems

File: install/food_del_robot_description/share/food_del_robot_description/urdf/common_properties.xacro (robot description, xacro)
@@ -1,38 +1 @@
-<?xml version="1.0"?>
-<robot xmlns:xacro="http://www.ros.org/wiki/xacro">
-    <!-- Materials -->
-    <material name="blue">
-        <color rgba="0.0 0.0 0.5 1.0"/>
-    </material>
-    <material name="red">
-        <color rgba="0.5 0.0 0.0 1.0"/>
-    </material>
-    <material name="green">
-        <color rgba="0.0 0.5 0.0 1.0"/>
-    </material>
-    <material name="black">
-        <color rgba="0.0 0.0 0.0 1.0"/>
-    </material>
-    <!-- Inertia -->
-    <xacro:macro name = "box_inertia" params = "m x y z o_xyz o_rpy">
-        <inertial>
-            <mass value="${m}"/>
-            <origin xyz="${o_xyz}" rpy="${o_rpy}"/>
-            <inertia ixx="${(m/12) * (y*y + z*z)}" ixy="0.0" ixz="0.0" iyy="${(m/12) * (x*x + z*z)}" iyz="0.0" izz="${(m/12) * (y*y + x*x)}"/>
-        </inertial>
-    </xacro:macro>
-    <xacro:macro name = "cylinder_inertia" params = "m r l o_xyz o_rpy">
-        <inertial>
-            <mass value="${m}"/>
-            <origin xyz="${o_xyz}" rpy="${o_rpy}"/>
-            <inertia ixx="${(m/12) * (3*r*r + l*l)}" ixy="0.0" ixz="0.0" iyy="${(m/12) * (3*r*r + l*l)}" iyz="0.0" izz="${(1/2) * m * r * r}"/>
-        </inertial>
-    </xacro:macro>
-    <xacro:macro name = "sphere_inertia" params = "m r o_xyz o_rpy">
-        <inertial>
-            <mass value="${m}"/>
-            <origin xyz="${o_xyz}" rpy="${o_rpy}"/>
-            <inertia ixx="${(2/5) * m * r * r}" ixy="0.0" ixz="0.0" iyy="${(2/5) * m * r * r}" iyz="0.0" izz="${(2/5) * m * r * r}"/>
-        </inertial>
-    </xacro:macro>
-</robot>
+/home/tikea/Food_Delivery_Robot/src/food_del_robot_description/urdf/common_properties.xacro

File: install/food_del_robot_description/share/food_del_robot_description/urdf/food_del_robot.ros2_control.xacro (robot description, xacro)
@@ -1,19 +1 @@
-<?xml version="1.0"?>
-<robot xmlns:xacro="http://www.ros.org/wiki/xacro">
-    <ros2_control name="FoodDeliveryRobotHardwareInterface" type="system">
-        <hardware>
-            <plugin>mock_components/GenericSystem</plugin>
-            <param name="calculate_dynamics">true</param>
-        </hardware>
-        <joint name="base_right_wheel_joint">
-            <command_interface name="velocity" />
-            <state_interface name="position" />
-            <state_interface name="velocity" />
-        </joint>
-        <joint name="base_left_wheel_joint">
-            <command_interface name="velocity" />
-            <state_interface name="position" />
-            <state_interface name="velocity" />
-        </joint>
-    </ros2_control>
-</robot>
+/home/tikea/Food_Delivery_Robot/src/food_del_robot_description/urdf/food_del_robot.ros2_control.xacro

File: install/food_del_robot_description/share/food_del_robot_description/urdf/food_del_robot.xacro (robot description, xacro)
@@ -1,152 +1 @@
-<?xml version="1.0"?>
-<robot name="food_del_robot" xmlns:xacro="http://www.ros.org/wiki/xacro">
-    <!-- Xacro parameters -->
-    <xacro:property name="base_length" value="0.48"/>
-    <xacro:property name="base_height" value="0.2"/>
-    <xacro:property name="base_width" value="0.48"/>
-    <xacro:property name="base_height_from_ground" value="0.01"/>
-    <xacro:property name="base_to_wheel_center" value="0.0555"/>
-    <xacro:property name="distance_between_two_wheels" value="0.45"/>
-    <xacro:property name="wheel_radius" value="0.065"/>
-    <xacro:property name="wheel_length" value="0.04"/>
-    <xacro:property name="rotate_90" value="1.57"/>
-    <xacro:property name ="lidar_length" value = "0.043"/>
-    <xacro:property name ="lidar_radius" value = "0.035"/>
-    <xacro:property name ="lidar_shift_from_center" value = "0.172"/>
-    <xacro:property name="imu_length" value="0.031"/>
-    <xacro:property name="imu_height" value="0.016"/>
-    <xacro:property name="imu_width" value="0.025"/>
-    <xacro:property name="imu_height_from_ground" value="0.110"/>
-    <!-- Wheel macro -->
-    <xacro:macro name="wheel_link" params="prefix">
-        <link name="${prefix}_wheel_link">
-            <visual>
-                <geometry>
-                    <cylinder radius="${wheel_radius}" length="${wheel_length}"/>
-                </geometry>
-                <!-- Rotate cylinder to roll correctly along Y axis -->
-                <origin xyz="0.0 0.0 0.0" rpy="${rotate_90} 0.0 0.0"/>
-                <material name="red"/>
-            </visual>
-            <collision>
-                <geometry>
-                    <sphere radius="${wheel_radius}"/>
-                </geometry>
-                <origin xyz="0.0 0.0 0.0" rpy="0.0 0.0 0.0"/>
-            </collision>
-            <xacro:cylinder_inertia
-                m="1.0"
-                r="${wheel_radius}"
-                l="${wheel_length}"
-                o_xyz="0.0 0.0 0.0"
-                o_rpy="0.0 ${rotate_90} 0.0"/>
-        </link>
-    </xacro:macro>
-    <!-- Instantiate wheels -->
-    <xacro:wheel_link prefix="right"/>
-    <xacro:wheel_link prefix="left"/>
-    <!-- Base footprint -->
-    <link name="base_footprint"/>
-    <!-- Base links -->
-    <link name="base_link">
-        <visual>
-            <geometry>
-                <box size="${base_length} ${base_width} ${base_height}"/>
-            </geometry>
-            <origin xyz="0.0 0.0 ${base_height / 2.0}" rpy="0.0 0.0 0.0"/>
-            <material name="blue"/>
-        </visual>
-        <collision>
-            <geometry>
-                <box size="${base_length} ${base_width} ${base_height}"/>
-            </geometry>
-            <origin xyz="0.0 0.0 ${base_height / 2.0}" rpy="0.0 0.0 0.0"/>
-        </collision>
-        <xacro:box_inertia
-            m="5.0"
-            x="${base_length}"
-            y="${base_width}"
-            z="${base_height}"
-            o_xyz="0.0 0.0 ${base_height / 2.0}"
-            o_rpy="0.0 0.0 0.0"/>
-    </link>
-    <!-- Base scan link -->
-    <link name="laser_link">
-        <visual>
-            <geometry>
-                <cylinder radius="${lidar_radius}" length="${lidar_length}"/>
-            </geometry>
-            <origin xyz="0.0 0.0 0.0" rpy="0.0 0.0 0.0"/>
-            <material name="black"/>
-        </visual>
-        <collision>
-            <geometry>
-                <cylinder radius="${lidar_radius}" length="${lidar_length}"/>
-            </geometry>
-            <origin xyz="0.0 0.0 0.0" rpy="0.0 0.0 0.0"/>
-        </collision>
-        <xacro:cylinder_inertia
-            m="0.2"
-            r="${lidar_radius}"
-            l="${lidar_length}"
-            o_xyz="0.0 0.0 0.0"
-            o_rpy="0.0 0.0 0.0"/>
-    </link>
-    <!-- IMU link -->
-    <link name="imu_link">
-        <visual>
-            <geometry>
-                <box size="${imu_length} ${imu_width} ${imu_height}"/>
-            </geometry>
-            <origin xyz="0.0 0.0 ${imu_height / 2.0}" rpy="0.0 0.0 0.0"/>
-            <material name="blue"/>
-        </visual>
-        <collision>
-            <geometry>
-                <box size="${imu_length} ${imu_width} ${imu_height}"/>
-            </geometry>
-            <origin xyz="0.0 0.0 ${imu_height / 2.0}" rpy="0.0 0.0 0.0"/>
-        </collision>
-        <xacro:box_inertia
-            m="5.0"
-            x="${imu_length}"
-            y="${imu_width}"
-            z="${imu_height}"
-            o_xyz="0.0 0.0 ${imu_height / 2.0}"
-            o_rpy="0.0 0.0 0.0"/>
-    </link>
-    <!-- base footprint - base link joint -->
-    <joint name="base_footprint_base_link_joint" type="fixed">
-        <origin xyz="0.0 0.0 ${base_height_from_ground}" rpy="0.0 0.0 0.0"/>
-        <parent link="base_footprint"/>
-        <child link="base_link"/>
-    </joint>
-    <!-- base link - right wheel link joint -->
-    <joint name="base_right_wheel_joint" type="revolute">
-        <origin xyz="0.0 ${distance_between_two_wheels/2} ${base_to_wheel_center}" rpy="0.0 0.0 0.0"/>
-        <parent link="base_link"/>
-        <child link="right_wheel_link"/>
-        <axis xyz="0.0 1.0 0.0"/>
-        <limit lower="0.0" upper="6.28" effort="100.0" velocity="5.0"/>
-    </joint>
-    <!-- base link - left wheel link joint -->
-    <joint name="base_left_wheel_joint" type="revolute">
-        <origin xyz="0.0 ${-distance_between_two_wheels/2} ${base_to_wheel_center}" rpy="0.0 0.0 0.0"/>
-        <parent link="base_link"/>
-        <child link="left_wheel_link"/>
-        <axis xyz="0.0 1.0 0.0"/>
-        <limit lower="0.0" upper="6.28" effort="100.0" velocity="5.0"/>
-    </joint>
-    <!-- base link - base scan link joint -->
-    <joint name="laser_base_link_joint" type="fixed">
-        <origin xyz="${lidar_shift_from_center} 0.0 ${base_height + (lidar_length/2)}" rpy="0.0 0.0 0.0"/>
-        <parent link="base_link"/>
-        <child link="laser_link"/>
-    </joint>
-    <!-- base link - imu link joint -->
-    <joint name="base_imu_joint" type="fixed">
-        <origin xyz="0.0 0.0 ${imu_height_from_ground}" rpy="0.0 0.0 0.0"/>
-        <parent link="base_link"/>
-        <child link="imu_link"/>
-    </joint>
-</robot>
+/home/tikea/Food_Delivery_Robot/src/food_del_robot_description/urdf/food_del_robot.xacro

File: install/food_del_robot_description/share/food_del_robot_description/urdf/food_del_robot_gazebo.xacro (robot description, xacro)
@@ -1,31 +1 @@
-<?xml version="1.0"?>
-<robot xmlns:xacro="http://www.ros.org/wiki/xacro">
-  <gazebo reference="front_caster_wheel_link">
-    <mu1>0.1</mu1>
-    <mu2>0.1</mu2>
-  </gazebo>
-  <gazebo reference="back_caster_wheel_link">
-    <mu1>0.1</mu1>
-    <mu2>0.1</mu2>
-  </gazebo>
-  <gazebo>
-    <plugin
-      filename="gz-sim-diff-drive-system"
-      name="gz::sim::systems::DiffDrive">
-      <left_joint>base_left_wheel_joint</left_joint>
-      <right_joint>base_right_wheel_joint</right_joint>
-      <wheel_separation>0.539</wheel_separation>
-      <wheel_radius>0.0695</wheel_radius>
-      <frame_id>odom</frame_id>
-      <child_frame_id>base_footprint</child_frame_id>
-    </plugin>
-  </gazebo>
-  <gazebo>
-    <plugin
-      filename="gz-sim-joint-state-publisher-system"
-      name="gz::sim::systems::JointStatePublisher">
-      <joint_name>base_left_wheel_joint</joint_name>
-      <joint_name>base_right_wheel_joint</joint_name>
-    </plugin>
-  </gazebo>
-</robot>
+/home/tikea/Food_Delivery_Robot/src/food_del_robot_description/urdf/food_del_robot_gazebo.xacro

File: install/food_del_robot_description/share/food_del_robot_description/urdf/my_main.urdf.xacro (robot description, xacro)
@@ -1,7 +1 @@
-<?xml version="1.0"?>
-<robot name="food_del_robot" xmlns:xacro="http://www.ros.org/wiki/xacro">
-    <xacro:include filename="common_properties.xacro"/>
-    <!-- <xacro:include filename="food_del_robot_gazebo.xacro"/> -->
-    <xacro:include filename="food_del_robot.xacro"/>
-    <xacro:include filename="food_del_robot.ros2_control.xacro"/>
-</robot>
+/home/tikea/Food_Delivery_Robot/src/food_del_robot_description/urdf/my_main.urdf.xacro

File: src/food_del_robot_description/urdf/food_del_robot.ros2_control.xacro (robot description, xacro)
@@ -1,8 +1,9 @@
 <?xml version="1.0"?>
 <robot xmlns:xacro="http://www.ros.org/wiki/xacro">
-    <ros2_control name="FoodDeliveryRobotHardwareInterface" type="system">
+    <ros2_control name="FoodDeliveryRobot" type="system">
         <hardware>
             <plugin>mock_components/GenericSystem</plugin>
             <param name="calculate_dynamics">true</param>
+            <!-- <plugin>food_del_robot_hardware/FoodDelRobotHardwareInterface</plugin> -->
         </hardware>
         <joint name="base_right_wheel_joint">
