Commit message: changed the joint type to continuous

File: src/food_del_robot_description/urdf/food_del_robot.ros2_control.xacro (robot description, xacro)
@@ -3,17 +3,17 @@
     <ros2_control name="FoodDeliveryRobot" type="system">
         <hardware>
-            <plugin>mock_components/GenericSystem</plugin>
-            <param name="calculate_dynamics">true</param>
-            <!-- <plugin>food_del_robot_hardware/FoodDelRobotHardwareInterface</plugin> -->
+            <!-- <plugin>mock_components/GenericSystem</plugin>
+            <param name="calculate_dynamics">true</param> -->
+            <plugin>food_del_robot_hardware/FoodDelRobotHardwareInterface</plugin>
         </hardware>
+        <joint name="base_left_wheel_joint">
+            <command_interface name="velocity"/>
+            <state_interface name="position"/>
+            <state_interface name="velocity"/>
+        </joint>
         <joint name="base_right_wheel_joint">
-            <command_interface name="velocity" />
-            <state_interface name="position" />
-            <state_interface name="velocity" />
-        </joint>
-        <joint name="base_left_wheel_joint">
-            <command_interface name="velocity" />
-            <state_interface name="position" />
-            <state_interface name="velocity" />
+            <command_interface name="velocity"/>
+            <state_interface name="position"/>
+            <state_interface name="velocity"/>
         </joint>
     </ros2_control>

File: src/food_del_robot_description/urdf/food_del_robot.xacro (robot description, xacro)
@@ -123,18 +123,16 @@
     </joint>
     <!-- base link - right wheel link joint -->
-    <joint name="base_right_wheel_joint" type="revolute">
+    <joint name="base_right_wheel_joint" type="continuous">
         <origin xyz="0.0 ${distance_between_two_wheels/2} ${base_to_wheel_center}" rpy="0.0 0.0 0.0"/>
         <parent link="base_link"/>
         <child link="right_wheel_link"/>
         <axis xyz="0.0 1.0 0.0"/>
-        <limit lower="0.0" upper="6.28" effort="100.0" velocity="5.0"/>
     </joint>
     <!-- base link - left wheel link joint -->
-    <joint name="base_left_wheel_joint" type="revolute">
+    <joint name="base_left_wheel_joint" type="continuous">
         <origin xyz="0.0 ${-distance_between_two_wheels/2} ${base_to_wheel_center}" rpy="0.0 0.0 0.0"/>
         <parent link="base_link"/>
         <child link="left_wheel_link"/>
         <axis xyz="0.0 1.0 0.0"/>
-        <limit lower="0.0" upper="6.28" effort="100.0" velocity="5.0"/>
     </joint>
     <!-- base link - base scan link joint -->
