Commit message: Added Camera into URDF, launch file for display the urdf of the robot, Fix the costmap problems and Added tf2_dynamics for wheel

File: src/food_del_robot_description/urdf/common_properties.xacro (robot description, xacro)
@@ -13,4 +13,7 @@
     <material name="black">
         <color rgba="0.0 0.0 0.0 1.0"/>
+    </material>
+    <material name="pink">
+        <color rgba="1.0 0.75 0.8 1.0"/>
     </material>
     <!-- Inertia -->

File: src/food_del_robot_description/urdf/food_del_robot.xacro (robot description, xacro)
@@ -18,4 +18,8 @@
     <xacro:property name="imu_width" value="0.025"/>
     <xacro:property name="imu_height_from_ground" value="0.110"/>
+    <xacro:property name="camera_length" value="0.025"/>
+    <xacro:property name="camera_height" value="0.025"/>
+    <xacro:property name="camera_width" value="0.09"/>
+    <xacro:property name="camera_height_from_ground" value="0.150"/>
     <!-- Wheel macro -->
     <xacro:macro name="wheel_link" params="prefix">
@@ -116,4 +120,27 @@
             o_rpy="0.0 0.0 0.0"/>
     </link>
+    <!-- Camera link -->
+    <link name="camera_link">
+        <visual>
+            <geometry>
+                <box size="${camera_length} ${camera_width} ${camera_height}"/>
+            </geometry>
+            <origin xyz="0.0 0.0 ${camera_height / 2.0}" rpy="0.0 0.0 0.0"/>
+            <material name="pink"/>
+        </visual>
+        <collision>
+            <geometry>
+                <box size="${camera_length} ${camera_width} ${camera_height}"/>
+            </geometry>
+            <origin xyz="0.0 0.0 ${camera_height / 2.0}" rpy="0.0 0.0 0.0"/>
+        </collision>
+        <xacro:box_inertia
+            m="0.5"
+            x="${camera_length}"
+            y="${camera_width}"
+            z="${camera_height}"
+            o_xyz="0.0 0.0 ${camera_height / 2.0}"
+            o_rpy="0.0 0.0 0.0"/>
+    </link>
     <!-- base footprint - base link joint -->
     <joint name="base_footprint_base_link_joint" type="fixed">
@@ -148,3 +175,9 @@
         <child link="imu_link"/>
     </joint>
+    <!-- base link - camera link joint -->
+    <joint name="base_camera_joint" type="fixed">
+        <origin xyz="${base_length/2.0} 0.0 ${camera_height_from_ground}" rpy="0.0 0.0 0.0"/>
+        <parent link="base_link"/>
+        <child link="camera_link"/>
+    </joint>
 </robot>

Commit message: added sim launch

File: src/food_del_robot_description/urdf/common_properties.xacro (robot description, xacro)
@@ -17,24 +17,32 @@
         <color rgba="1.0 0.75 0.8 1.0"/>
     </material>
-    <!-- Inertia -->
-    <xacro:macro name = "box_inertia" params = "m x y z o_xyz o_rpy">
+    <material name="gray">
+        <color rgba="0.5 0.5 0.5 1"/>
+    </material>
+    <xacro:macro name="box_inertia" params="m l w h xyz rpy">
         <inertial>
+            <origin xyz="${xyz}" rpy="${rpy}"/>
             <mass value="${m}"/>
-            <origin xyz="${o_xyz}" rpy="${o_rpy}"/>
-            <inertia ixx="${(m/12) * (y*y + z*z)}" ixy="0.0" ixz="0.0" iyy="${(m/12) * (x*x + z*z)}" iyz="0.0" izz="${(m/12) * (y*y + x*x)}"/>
+            <inertia ixx="${(1/12.0) * m * (h*h + l*l)}" ixy="0" ixz="0"
+                     iyy="${(1/12.0) * m * (w*w + l*l)}" iyz="0"
+                     izz="${(1/12.0) * m * (w*w + h*h)}"/>
         </inertial>
     </xacro:macro>
-    <xacro:macro name = "cylinder_inertia" params = "m r l o_xyz o_rpy">
+    <xacro:macro name="cylinder_inertia" params="m r h xyz rpy">
         <inertial>
+            <origin xyz="${xyz}" rpy="${rpy}"/>
             <mass value="${m}"/>
-            <origin xyz="${o_xyz}" rpy="${o_rpy}"/>
-            <inertia ixx="${(m/12) * (3*r*r + l*l)}" ixy="0.0" ixz="0.0" iyy="${(m/12) * (3*r*r + l*l)}" iyz="0.0" izz="${(1/2) * m * r * r}"/>
+            <inertia ixx="${(1/12.0) * m * (3*r*r + h*h)}" ixy="0" ixz="0"
+                     iyy="${(1/12.0) * m * (3*r*r + h*h)}" iyz="0"
+                     izz="${0.5 * m * r*r}"/>
         </inertial>
     </xacro:macro>
-    <xacro:macro name = "sphere_inertia" params = "m r o_xyz o_rpy">
+    <xacro:macro name="sphere_inertia" params="m r xyz rpy">
         <inertial>
+            <origin xyz="${xyz}" rpy="${rpy}"/>
             <mass value="${m}"/>
-            <origin xyz="${o_xyz}" rpy="${o_rpy}"/>
-            <inertia ixx="${(2/5) * m * r * r}" ixy="0.0" ixz="0.0" iyy="${(2/5) * m * r * r}" iyz="0.0" izz="${(2/5) * m * r * r}"/>
+            <inertia ixx="${(2/5.0) * m * r*r}" ixy="0" ixz="0"
+                     iyy="${(2/5.0) * m * r*r}" iyz="0"
+                     izz="${(2/5.0) * m * r*r}"/>
         </inertial>
     </xacro:macro>
