Commit message: Update STVL layer in Simulation and fix major issues

File: src/food_del_robot_description/urdf/food_del_robot.urdf.xacro (robot description, xacro)
@@ -166,9 +166,23 @@
     </collision>
   </link>
+  <!-- FIXED: raise camera and tilt it upward a bit -->
   <joint name="camera_base_joint" type="fixed">
-    <origin xyz="0.29541 0.0175 0.168" rpy="0 0 0"/>
+    <origin xyz="0.29541 0.0175 0.23" rpy="0 -0.35 0"/>
     <parent link="base_link"/>
     <child link="camera_link"/>
     <axis xyz="0 0 0"/>
+  </joint>
+  <!-- Added camera frames for ROS optical convention -->
+  <link name="camera_rgb_frame"/>
+  <joint name="camera_rgb_joint" type="fixed">
+    <origin xyz="0 0 0" rpy="0 0 0"/>
+    <parent link="camera_link"/>
+    <child link="camera_rgb_frame"/>
+  </joint>
+  <link name="camera_rgb_optical_frame"/>
+  <joint name="camera_rgb_optical_joint" type="fixed">
+    <origin xyz="0 0 0" rpy="-1.57079632679 0 -1.57079632679"/>
+    <parent link="camera_rgb_frame"/>
+    <child link="camera_rgb_optical_frame"/>
   </joint>
   <link name="imu_link">
@@ -334,5 +348,5 @@
             </horizontal>
           </scan>
-          <range><min>0.1</min><max>12</max></range>
+          <range><min>0.2</min><max>12</max></range>
         </ray>
         <plugin name="lidar" filename="libgazebo_ros_ray_sensor.so">
@@ -347,4 +361,40 @@
       </sensor>
     </gazebo>
+    <!-- RGB-D camera for RTAB-Map + PointCloud2 for STVL -->
+    <gazebo reference="camera_link">
+      <sensor name="camera" type="depth">
+        <pose>0 0 0 0 0 0</pose>
+        <visualize>true</visualize>
+        <update_rate>15</update_rate>      <!-- reduced from 30, enough for obstacle detection -->
+        <camera>
+          <horizontal_fov>1.047198</horizontal_fov>
+          <image>
+            <width>640</width>
+            <height>480</height>
+            <format>R8G8B8</format>
+          </image>
+          <clip>
+            <near>0.1</near>
+            <far>5.0</far>
+          </clip>
+        </camera>
+        <plugin name="camera_controller" filename="libgazebo_ros_camera.so">
+          <frame_name>camera_rgb_optical_frame</frame_name>
+          <camera_name>camera</camera_name>
+          <hack_baseline>0.0</hack_baseline>
+          <min_depth>0.1</min_depth>
+          <max_depth>5.0</max_depth>
+          <ros>
+            <namespace>/</namespace>
+            <remapping>~/image_raw:=camera/image_raw</remapping>
+            <remapping>~/depth_image:=cdepth/points</remapping>   <!-- ADD THIS -->
+          </ros>
+          <!-- ADD THESE — enables PointCloud2 publishing directly -->
+          <point_cloud_topic>camera/depth/points</point_cloud_topic>
+          <point_cloud_cutoff>0.1</point_cloud_cutoff>
+          <point_cloud_cutoff_max>5.0</point_cloud_cutoff_max>
+        </plugin>
+      </sensor>
+    </gazebo>
   </xacro:if>
 </robot>

Commit message: implement real camera and lidar to the urdf file

File: src/food_del_robot_description/urdf/food_del_robot.urdf.xacro (robot description, xacro)
@@ -2,5 +2,4 @@
 <robot name="food_del_robot"
   xmlns:xacro="http://www.ros.org/wiki/xacro">
-  <!-- Pass use_sim:=true from launch file to activate Gazebo plugins -->
   <xacro:arg name="use_sim" default="false"/>
   <!-- ============================================================
@@ -34,5 +33,4 @@
     </inertial>
   </xacro:macro>
-  <!-- Wheel spinning about Y axis -->
   <xacro:macro name="wheel_inertia" params="m r h xyz rpy">
     <inertial>
@@ -122,4 +120,8 @@
     <axis xyz="0 1 0"/>
   </joint>
+  <!-- ============================================================
+       LiDAR — RPLidar A1
+       360° scan, 0.15m–12m, 1° resolution = 360 samples
+       ============================================================ -->
   <link name="lidar_link">
     <xacro:box_inertia m="0.01" l="0.1" w="0.1" h="0.02"
@@ -147,6 +149,12 @@
     <axis xyz="0 0 0"/>
   </joint>
+  <!-- ============================================================
+       Camera — Intel RealSense D435i
+       Depth FOV: 87°x58°, Range: 0.3m–3m
+       RGB: 1920x1080 @ 30fps
+       ============================================================ -->
   <link name="camera_link">
-    <xacro:box_inertia m="0.01" l="0.05" w="0.03" h="0.03"
+    <!-- D435i real dimensions: 90mm x 25mm x 25mm -->
+    <xacro:box_inertia m="0.072" l="0.09" w="0.025" h="0.025"
                        xyz="0 0 0" rpy="0 0 0"/>
     <visual>
@@ -162,9 +170,9 @@
       <origin xyz="0 0 0" rpy="0 0 0"/>
       <geometry>
-        <box size="0.05 0.03 0.03"/>
-      </geometry>
-    </collision>
-  </link>
-  <!-- FIXED: raise camera and tilt it upward a bit -->
+        <!-- D435i actual size -->
+        <box size="0.09 0.025 0.025"/>
+      </geometry>
+    </collision>
+  </link>
   <joint name="camera_base_joint" type="fixed">
     <origin xyz="0.29541 0.0175 0.23" rpy="0 -0.35 0"/>
@@ -173,5 +181,5 @@
     <axis xyz="0 0 0"/>
   </joint>
-  <!-- Added camera frames for ROS optical convention -->
+  <!-- ROS optical convention frames for D435i -->
   <link name="camera_rgb_frame"/>
   <joint name="camera_rgb_joint" type="fixed">
@@ -186,4 +194,18 @@
     <child link="camera_rgb_optical_frame"/>
   </joint>
+  <!-- Depth optical frame for D435i pointcloud -->
+  <link name="camera_depth_frame"/>
+  <joint name="camera_depth_joint" type="fixed">
+    <origin xyz="0 0 0" rpy="0 0 0"/>
+    <parent link="camera_link"/>
+    <child link="camera_depth_frame"/>
+  </joint>
+  <link name="camera_depth_optical_frame"/>
+  <joint name="camera_depth_optical_joint" type="fixed">
+    <origin xyz="0 0 0" rpy="-1.57079632679 0 -1.57079632679"/>
+    <parent link="camera_depth_frame"/>
+    <child link="camera_depth_optical_frame"/>
+  </joint>
+  <!-- IMU link -->
   <link name="imu_link">
     <xacro:box_inertia m="0.01" l="0.01" w="0.01" h="0.01"
@@ -211,15 +233,12 @@
     <axis xyz="0 0 0"/>
   </joint>
+  <!-- Caster wheels (unchanged) -->
   <link name="caster1_link">
     <xacro:sphere_inertia m="0.108" r="0.0325" xyz="0 0 0" rpy="0 0 0"/>
-    <visual>
-      <origin xyz="0 0 0" rpy="0 0 0"/>
-      <geometry>
-        <mesh filename="package://food_del_robot_description/meshes/caster1_link.STL"/>
-      </geometry>
+    <visual><origin xyz="0 0 0" rpy="0 0 0"/>
+      <geometry><mesh filename="package://food_del_robot_description/meshes/caster1_link.STL"/></geometry>
       <material name=""><color rgba="0.75 0.75 0.75 1"/></material>
     </visual>
-    <collision>
-      <origin xyz="0 0 0" rpy="0 0 0"/>
+    <collision><origin xyz="0 0 0" rpy="0 0 0"/>
       <geometry><sphere radius="0.0325"/></geometry>
     </collision>
@@ -232,13 +251,9 @@
   <link name="caster2_link">
     <xacro:sphere_inertia m="0.108" r="0.0325" xyz="0 0 0" rpy="0 0 0"/>
-    <visual>
-      <origin xyz="0 0 0" rpy="0 0 0"/>
-      <geometry>
-        <mesh filename="package://food_del_robot_description/meshes/caster2_link.STL"/>
-      </geometry>
+    <visual><origin xyz="0 0 0" rpy="0 0 0"/>
+      <geometry><mesh filename="package://food_del_robot_description/meshes/caster2_link.STL"/></geometry>
       <material name=""><color rgba="0.75 0.75 0.75 1"/></material>
     </visual>
-    <collision>
-      <origin xyz="0 0 0" rpy="0 0 0"/>
+    <collision><origin xyz="0 0 0" rpy="0 0 0"/>
       <geometry><sphere radius="0.0325"/></geometry>
     </collision>
@@ -251,13 +266,9 @@
   <link name="caster3_link">
     <xacro:sphere_inertia m="0.108" r="0.0325" xyz="0 0 0" rpy="0 0 0"/>
-    <visual>
-      <origin xyz="0 0 0" rpy="0 0 0"/>
-      <geometry>
-        <mesh filename="package://food_del_robot_description/meshes/caster3_link.STL"/>
-      </geometry>
+    <visual><origin xyz="0 0 0" rpy="0 0 0"/>
+      <geometry><mesh filename="package://food_del_robot_description/meshes/caster3_link.STL"/></geometry>
       <material name=""><color rgba="0.75 0.75 0.75 1"/></material>
     </visual>
-    <collision>
-      <origin xyz="0 0 0" rpy="0 0 0"/>
+    <collision><origin xyz="0 0 0" rpy="0 0 0"/>
       <geometry><sphere radius="0.0325"/></geometry>
     </collision>
@@ -270,13 +281,9 @@
   <link name="caster4_link">
     <xacro:sphere_inertia m="0.108" r="0.0325" xyz="0 0 0" rpy="0 0 0"/>
-    <visual>
-      <origin xyz="0 0 0" rpy="0 0 0"/>
-      <geometry>
-        <mesh filename="package://food_del_robot_description/meshes/caster4_link.STL"/>
-      </geometry>
+    <visual><origin xyz="0 0 0" rpy="0 0 0"/>
+      <geometry><mesh filename="package://food_del_robot_description/meshes/caster4_link.STL"/></geometry>
       <material name=""><color rgba="0.75 0.75 0.75 1"/></material>
     </visual>
-    <collision>
-      <origin xyz="0 0 0" rpy="0 0 0"/>
+    <collision><origin xyz="0 0 0" rpy="0 0 0"/>
       <geometry><sphere radius="0.0325"/></geometry>
     </collision>
@@ -288,5 +295,5 @@
   </joint>
   <!-- ============================================================
-       Gazebo simulation — only loaded when use_sim:=true
+       Gazebo plugins — only loaded when use_sim:=true
        ============================================================ -->
   <xacro:if value="$(arg use_sim)">
@@ -302,5 +309,5 @@
       <minDepth>0.001</minDepth><maxVel>0.1</maxVel>
     </gazebo>
-    <!-- Caster friction (low to allow free rolling) -->
+    <!-- Caster friction -->
     <gazebo reference="caster1_link">
       <mu1>0.01</mu1><mu2>0.01</mu2><kp>100000.0</kp><kd>100.0</kd>
@@ -315,5 +322,5 @@
       <mu1>0.01</mu1><mu2>0.01</mu2><kp>100000.0</kp><kd>100.0</kd>
     </gazebo>
-    <!-- Differential drive plugin -->
+    <!-- Differential drive plugin (unchanged) -->
     <gazebo>
       <plugin filename="libgazebo_ros_diff_drive.so" name="diff_drive_controller">
@@ -333,20 +340,33 @@
       </plugin>
     </gazebo>
-    <!-- LiDAR ray sensor -->
+    <!-- =====================================================
+         RPLidar A1 — Ray sensor
+         360°, 0.15m–12m, 1° resolution = 360 samples
+         Scan rate: 5.5Hz (use 8Hz as safe upper sim value)
+         ===================================================== -->
     <gazebo reference="lidar_link">
       <sensor name="lidar" type="ray">
         <pose>0 0 0 0 0 0</pose>
         <visualize>true</visualize>
-        <update_rate>8</update_rate>
+        <update_rate>5.5</update_rate>        <!-- RPLidar A1 typical scan rate -->
         <ray>
           <scan>
             <horizontal>
-              <samples>1083</samples>
+              <samples>360</samples>          <!-- 1° resolution = 360 samples for full 360° -->
               <resolution>1</resolution>
-              <min_angle>-3.1241390705108643</min_angle>
-              <max_angle>3.1415927410125732</max_angle>
+              <min_angle>-3.14159265</min_angle>   <!-- -180° full 360° scan -->
+              <max_angle>3.14159265</max_angle>    <!-- +180° -->
             </horizontal>
           </scan>
-          <range><min>0.2</min><max>12</max></range>
+          <range>
+            <min>0.15</min>                   <!-- RPLidar A1 min range -->
+            <max>12.0</max>                   <!-- RPLidar A1 max range -->
+            <resolution>0.002</resolution>    <!-- 0.2cm distance resolution -->
+          </range>
+          <noise>
+            <type>gaussian</type>
+            <mean>0.0</mean>
+            <stddev>0.01</stddev>             <!-- ~1cm noise typical for A1 -->
+          </noise>
         </ray>
         <plugin name="lidar" filename="libgazebo_ros_ray_sensor.so">
@@ -357,41 +377,51 @@
           <topic>scan</topic>
           <frame_name>lidar_link</frame_name>
-          <transport>ros</transport>
         </plugin>
       </sensor>
     </gazebo>
-    <!-- RGB-D camera for RTAB-Map + PointCloud2 for STVL -->
+    <!-- =====================================================
+         Intel RealSense D435i
+         RGB:   1920x1080 @ 30fps, FOV 69.4°x42.5°
+         Depth: 1280x720  @ 30fps, FOV 87°x58°
+         Range: 0.3m – 3m (ideal), absolute min 0.105m
+         ===================================================== -->
     <gazebo reference="camera_link">
-      <sensor name="camera" type="depth">
+      <sensor name="d435i_camera" type="depth">
         <pose>0 0 0 0 0 0</pose>
         <visualize>true</visualize>
-        <update_rate>15</update_rate>      <!-- reduced from 30, enough for obstacle detection -->
+        <update_rate>30</update_rate>         <!-- D435i RGB: 30fps -->
         <camera>
-          <horizontal_fov>1.047198</horizontal_fov>
+          <!-- Depth FOV: 87°x58° → horizontal = 1.5184 rad, vertical = 1.0123 rad -->
+          <horizontal_fov>1.5184</horizontal_fov>   <!-- 87° in radians -->
+          <!-- Use depth resolution for obstacle detection -->
           <image>
-            <width>640</width>
-            <height>480</height>
+            <width>1280</width>               <!-- D435i depth resolution -->
+            <height>720</height>
             <format>R8G8B8</format>
           </image>
           <clip>
-            <near>0.1</near>
-            <far>5.0</far>
+            <near>0.3</near>                  <!-- D435i ideal min depth 0.3m -->
+            <far>3.0</far>                    <!-- D435i ideal max depth 3m -->
           </clip>
+          <noise>
+            <type>gaussian</type>
+            <mean>0.0</mean>
+            <stddev>0.005</stddev>            <!-- ~5mm depth noise typical for D435i -->
+          </noise>
         </camera>
-        <plugin name="camera_controller" filename="libgazebo_ros_camera.so">
-          <frame_name>camera_rgb_optical_frame</frame_name>
+        <plugin name="d435i_controller" filename="libgazebo_ros_camera.so">
+          <frame_name>camera_depth_optical_frame</frame_name>
           <camera_name>camera</camera_name>
           <hack_baseline>0.0</hack_baseline>
-          <min_depth>0.1</min_depth>
-          <max_depth>5.0</max_depth>
+          <min_depth>0.3</min_depth>          <!-- D435i ideal min -->
+          <max_depth>3.0</max_depth>          <!-- D435i ideal max -->
           <ros>
             <namespace>/</namespace>
             <remapping>~/image_raw:=camera/image_raw</remapping>
-            <remapping>~/depth_image:=cdepth/points</remapping>   <!-- ADD THIS -->
+            <remapping>~/depth_image:=camera/depth/image_raw</remapping>
           </ros>
-          <!-- ADD THESE — enables PointCloud2 publishing directly -->
           <point_cloud_topic>camera/depth/points</point_cloud_topic>
-          <point_cloud_cutoff>0.1</point_cloud_cutoff>
-          <point_cloud_cutoff_max>5.0</point_cloud_cutoff_max>
+          <point_cloud_cutoff>0.3</point_cloud_cutoff>      <!-- match min_depth -->
+          <point_cloud_cutoff_max>3.0</point_cloud_cutoff_max>
         </plugin>
       </sensor>
