Commit message: Fully update for simulation

File: src/food_del_robot_description/urdf/Real_Robot/food_del_robot.xacro (robot description, xacro)
@@ -27,8 +27,9 @@
             <visual>
                 <geometry>
-                    <cylinder radius="${wheel_radius}" length="${wheel_length}"/>
+                    <mesh filename="file:///home/panha/Food_Delivery_Robot/src/food_del_robot_description/urdf/Real_Robot/${prefix}_wheel_link.STL"
+                          scale="1 1 1"/>
                 </geometry>
-                <!-- Rotate cylinder to roll correctly along Y axis -->
-                <origin xyz="0.0 0.0 0.0" rpy="${rotate_90} 0.0 0.0"/>
+                <!-- Rotate wheel mesh to roll correctly along Y axis -->
+                <origin xyz="0.0 0.0 0.0" rpy="0.0 0.0 0.0"/>
                 <material name="red"/>
             </visual>
@@ -56,7 +57,8 @@
         <visual>
             <geometry>
-                <box size="${base_length} ${base_width} ${base_height}"/>
+                <mesh filename="file:///home/panha/Food_Delivery_Robot/src/food_del_robot_description/urdf/Real_Robot/base_link.STL"
+                    scale="1 1 1"/>
             </geometry>
-            <origin xyz="0.0 0.0 ${base_height / 2.0}" rpy="0.0 0.0 0.0"/>
+            <origin xyz="0.0 0.0 0.1" rpy="0.0 0.0 1.57"/>
             <material name="blue"/>
         </visual>

File: src/food_del_robot_description/urdf/Simulation/mobile_base_gazebo_sim.xacro (robot description, xacro)
@@ -30,13 +30,12 @@
     </gazebo>
     <gazebo reference="caster_wheel_real_link">
-        <material>Gazebo/Gray</material>
-        <mu1>1.5</mu1>
-        <mu2>1.5</mu2>
+        <mu1>0.0</mu1>   <!-- Should be near-zero for free-rolling -->
+        <mu2>0.0</mu2>
         <kp>1000000.0</kp>
         <kd>100.0</kd>
         <minDepth>0.001</minDepth>
-        <maxVel>0.1</maxVel>
-        <slip1>0.0</slip1>
-        <slip2>0.0</slip2>
+        <maxVel>1.0</maxVel>   <!-- Also increase this -->
+        <slip1>1.0</slip1>     <!-- Allow slip -->
+        <slip2>1.0</slip2>
     </gazebo>
     <gazebo reference="laser_link">
@@ -56,5 +55,5 @@
                 </scan>
                 <range>
-                    <min>0.5</min>
+                    <min>0.1</min>
                     <max>12</max>
                 </range>
@@ -72,9 +71,9 @@
     </gazebo>
     <gazebo>
-        <plugin name="diff_drive_controller" filename="libgazebo_ros_diff_drive.so">
+        <plugin filename="libgazebo_ros_diff_drive.so" name="diff_drive_controller">
             <update_rate>50</update_rate>
             <left_joint>base_left_wheel_joint</left_joint>
             <right_joint>base_right_wheel_joint</right_joint>
-            <wheel_separation>0.41</wheel_separation>
+            <wheel_separation>0.45</wheel_separation>
             <wheel_diameter>0.2</wheel_diameter>
             <publish_odom>true</publish_odom>

File: src/food_del_robot_description/urdf/Simulation/mobile_base_sim.xacro (robot description, xacro)
@@ -105,15 +105,13 @@
         <axis xyz="0 1 0"/>
     </joint>
-    <joint name="base_caster_wheel_support_joint" type="continuous">
+    <joint name="base_caster_wheel_support_joint" type="fixed">
         <parent link="base_link"/>
         <child link="caster_wheel_link_support"/>
         <origin xyz="${base_length / 3.0} 0 ${-caster_wheel_support_length / 2.0}" rpy="0 0 0"/>
-        <axis xyz="0 0 1"/>
     </joint>
-    <joint name="base_caster_wheel_real_joint" type="continuous">
+    <joint name="base_caster_wheel_real_joint" type="fixed">
         <parent link="caster_wheel_link_support"/>
         <child link="caster_wheel_real_link"/>
         <origin xyz="0 0 ${-caster_wheel_support_length / 2.0 - caster_wheel_real_radius}" rpy="1.57 1.57 0"/>
-        <axis xyz="0 0 1"/>
     </joint>
     <joint name="base_joint" type="fixed">
